File: PowerBoardRedux/powerboard redux.brd (EAGLE design)
At the start: 65 x 30 mm, 44 parts, among them CN1 microUSB, Q1 BSS138, SW1 1825027-5, T1 MMUN2133LT1G, U1 TPS61090RSAR, U2 MCP73871

Commit message: Managed to make board & schematic inconsistent, fixed
Routing:
- net VBAT: track 66.2 -> 69.4 mm
- net VBUS: track 83.9 -> 82.6 mm
- net LBO: track 45.8 -> 46.8 mm
Other:
- board text added: "PowerBoardRedux v1 2019 jdimpson From an AdaFruit design"
- board text removed: "PowerBoardRedux v1.01 2019 jdimpson From an AdaFruit design"

Commit message: Cleanup for BOM upload
Parts:
- renumbered LED1 to LOW, LED2 to PWR, U$11 to SW2
Changed lines of the file:
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@@
 <layer number="25" name="tNames" color="7" fill="1" visible="yes" active="yes"/>
 <layer number="26" name="bNames" color="7" fill="1" visible="yes" active="yes"/>
-<layer number="27" name="tValues" color="7" fill="1" visible="yes" active="yes"/>
-<layer number="28" name="bValues" color="7" fill="1" visible="yes" active="yes"/>
+<layer number="27" name="tValues" color="7" fill="1" visible="no" active="yes"/>
+<layer number="28" name="bValues" color="7" fill="1" visible="no" active="yes"/>
 <layer number="29" name="tStop" color="7" fill="3" visible="no" active="yes"/>
 <layer number="30" name="bStop" color="7" fill="6" visible="no" active="yes"/>
@@
 </element>
 <element name="B1" library="microbuilder" package="JSTPH2" value="JST 2-PH" x="58.42" y="12.827" smashed="yes" rot="R180">
-<attribute name="NAME" x="91.3715" y="50.3815" size="0.8128" layer="25" ratio="18" rot="R180"/>
+<attribute name="NAME" x="79.3065" y="32.2205" size="0.8128" layer="25" ratio="18" rot="R180"/>
 <attribute name="VALUE" x="86.8045" y="50.8" size="1.016" layer="27" font="vector" ratio="10" rot="R180"/>
 </element>
@@
 <attribute name="BOM" value="EXCLUDE" x="11.279" y="-18.946" size="1.778" layer="27" rot="R270" display="off"/>
 </element>
-<element name="LED1" library="microbuilder" package="CHIPLED_0805_NOOUTLINE" value="RED" x="63.659" y="11.27" smashed="yes" rot="R180">
+<element name="LOW" library="microbuilder" package="CHIPLED_0805_NOOUTLINE" value="RED" x="63.659" y="11.27" smashed="yes" rot="R180">
 <attribute name="VALUE" x="88.192" y="50.711" size="1.016" layer="27" font="vector" ratio="10" rot="R270"/>
 </element>
@@
 <attribute name="VALUE" x="77.375" y="10.6186" size="1.016" layer="27" font="vector" ratio="10" rot="R90"/>
 </element>
-<element name="LED2" library="microbuilder" package="CHIPLED_0805_NOOUTLINE" value="BLUE" x="41.089" y="32.544" smashed="yes" rot="R270">
+<element name="PWR" library="microbuilder" package="CHIPLED_0805_NOOUTLINE" value="BLUE" x="41.089" y="32.544" smashed="yes" rot="R270">
 <attribute name="VALUE" x="76.289" y="23.641" size="1.016" layer="27" font="vector" ratio="10"/>
 </element>
@@
 </element>
 <element name="JP2" library="microbuilder" package="1X08_ROUND" value="" x="23.749" y="19.558" smashed="yes" rot="R180">
-<attribute name="NAME" x="36.7792" y="54.6862" size="0.8128" layer="25" ratio="18" rot="R180"/>
+<attribute name="NAME" x="77.2922" y="33.8582" size="0.8128" layer="25" ratio="18" rot="R180"/>
 <attribute name="VALUE" x="33.909" y="22.733" size="0.4064" layer="27" ratio="10" rot="R180"/>
 </element>
@@
 <element name="SW1" library="right angle tactile switch 1825027-5 te connect" package="SW2_1825027-A" value="1825027-5" x="15.494" y="10.922" smashed="yes">
 <attribute name="MANUFACTURER_PART_NUMBER" value="18250275" x="11.303" y="29.21" size="1.778" layer="27" display="off"/>
-<attribute name="NAME" x="28.575" y="51.1302" size="1.27" layer="25" ratio="6" rot="SR0"/>
+<attribute name="NAME" x="73.279" y="36.3982" size="1.27" layer="25" ratio="6" rot="SR0"/>
 <attribute name="VENDOR" value="TE Connectivity" x="11.303" y="29.21" size="1.778" layer="27" display="off"/>
 </element>
 <element name="S4" library="SparkFun-Switches" library_urn="urn:adsk.eagle:library:535" package="TACTILE_SWITCH_PTH_6.0MM" package3d_urn="urn:adsk.eagle:package:40163/1" value="MOMENTARY-SWITCH-SPST-PTH-6.0MM" x="21.336" y="13.462" smashed="yes">
-<attribute name="NAME" x="40.513" y="54.229" size="0.6096" layer="25" font="vector" ratio="20" align="bottom-center"/>
+<attribute name="NAME" x="78.867" y="33.528" size="0.6096" layer="25" font="vector" ratio="20" align="bottom-center"/>
 <attribute name="PROD_ID" value=" SWCH-08441" x="17.018" y="-11.303" size="1.778" layer="27" display="off"/>
 <attribute name="SF_SKU" value="COM-00097" x="17.018" y="-11.303" size="1.778" layer="27" display="off"/>
@@
 </element>
 <element name="CN1" library="microusb-amphenol-10118194-0001LF" package="4UCONN_20329" value="microUSB" x="66.167" y="21.082" rot="R90"/>
-<element name="U$11" library="rightangleslideswitchspdt" package="OS102011MA1QN1" value="OS102011MA1QN1" x="8.509" y="23.241" rot="R270"/>
+<element name="SW2" library="rightangleslideswitchspdt" package="OS102011MA1QN1" value="OS102011MA1QN1" x="8.509" y="23.241" rot="R270"/>
 <element name="JP1" library="microbuilder" package="1X02_ROUND" value="JP1" x="58.42" y="11.811" smashed="yes">
-<attribute name="NAME" x="71.6788" y="55.8038" size="0.8128" layer="25" ratio="18"/>
+<attribute name="NAME" x="73.7108" y="33.4518" size="0.8128" layer="25" ratio="18"/>
 <attribute name="VALUE" x="80.772" y="50.927" size="0.4064" layer="27" ratio="10"/>
 </element>
@@
 <contactref element="C2" pad="2"/>
 <contactref element="R2" pad="1"/>
-<contactref element="LED1" pad="C"/>
+<contactref element="LOW" pad="C"/>
 <polygon width="0.254" layer="1" spacing="0.254" isolate="0.254" rank="2">
 <vertex x="71.12" y="39.37"/>
@@
 <vertex x="71.12" y="39.37"/>
 </polygon>
-<contactref element="LED2" pad="C"/>
+<contactref element="PWR" pad="C"/>
 <wire x1="45.792" y1="24.025" x2="45.792" y2="23.059" width="0.254" layer="1"/>
 <wire x1="45.792" y1="23.059" x2="45.593" y2="22.86" width="0.254" layer="1"/>
@@
 <wire x1="65.267" y1="18.544" x2="64.95" y2="18.227" width="0.4064" layer="1"/>
 <wire x1="64.95" y1="18.227" x2="61.976" y2="18.227" width="0.4064" layer="1"/>
-<contactref element="U$11" pad="P$1"/>
+<contactref element="SW2" pad="P$1"/>
 <wire x1="54.296" y1="10.22" x2="53.34" y2="11.176" width="0.2032" layer="1"/>
 <wire x1="53.34" y1="11.176" x2="53.34" y2="12.827" width="0.2032" layer="1"/>
@@
 <wire x1="51.816" y1="18.542" x2="50.6774" y2="19.6806" width="0.254" layer="16"/>
 <wire x1="50.6774" y1="19.6806" x2="50.6774" y2="22.5957875" width="0.254" layer="16"/>
-<contactref element="U$11" pad="P$3"/>
+<contactref element="SW2" pad="P$3"/>
 <wire x1="14.4366625" y1="17.3736" x2="12.5692625" y2="19.241" width="0.2032" layer="1"/>
 <wire x1="12.5692625" y1="19.241" x2="8.509" y2="19.241" width="0.2032" layer="1"/>
@@
 </signal>
 <signal name="N$2">
-<contactref element="LED1" pad="A"/>
+<contactref element="LOW" pad="A"/>
 <contactref element="R20" pad="1"/>
 <wire x1="53.245" y1="14.558" x2="54.214" y2="13.589" width="0.254" layer="1"/>
@@
 <contactref element="JP2" pad="4"/>
 <wire x1="49.902" y1="22.25" x2="49.944" y2="22.292" width="0.254" layer="1"/>
-<contactref element="U$11" pad="P$2"/>
+<contactref element="SW2" pad="P$2"/>
 <via x="49.944" y="22.292" extent="1-16" drill="0.4"/>
 <wire x1="8.509" y1="21.241" x2="11.144" y2="21.241" width="0.2032" layer="1"/>
@@
 <signal name="N$4">
 <contactref element="R5" pad="2"/>
-<contactref element="LED2" pad="A"/>
+<contactref element="PWR" pad="A"/>
 <wire x1="40.386" y1="26.985" x2="40.005" y2="26.985" width="0.254" layer="1"/>
 <wire x1="40.386" y1="26.985" x2="40.386" y2="28.43126875" width="0.254" layer="1"/>
