File: PowerBoardRedux/powerboard redux.sch (EAGLE design)
At the start: 44 parts, among them CN1 microUSB, Q1 BSS138, SW1 1825027-5, T1 MMUN2133LT1G, U1 TPS61090RSAR, U2 MCP73871

Commit message: Managed to make board & schematic inconsistent, fixed
Changed lines of the file:
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@@
 <part name="U$43" library="microbuilder" deviceset="VLIPO" device=""/>
 <part name="U2" library="microbuilder" deviceset="MCP73871" device="" value="MCP73871"/>
+<part name="U$13" library="microbuilder" deviceset="FRAME_A4_ADAFRUIT" device=""/>
 <part name="RPI1" library="microbuilder" deviceset="RASPBERRYPI_BPLUS" device="_BONNETNODIM" value="RASPBERRYPI_BPLUS_BONNETNODIM"/>
 <part name="GND3" library="supply1" deviceset="GND" device=""/>
@@
 <instance part="U$43" gate="G$1" x="73.66" y="99.06"/>
 <instance part="U2" gate="G$1" x="203.2" y="127"/>
+<instance part="U$13" gate="G$1" x="0" y="0"/>
 <instance part="RPI1" gate="G$1" x="33.02" y="142.24"/>
 <instance part="GND3" gate="1" x="55.88" y="109.22"/>
@@
 <pinref part="U$11" gate="G$1" pin="P$3"/>
 <wire x1="157.48" y1="60.96" x2="157.48" y2="50.8" width="0.1524" layer="91"/>
-<wire x1="157.48" y1="50.8" x2="170.18" y2="50.8" width="0.1524" layer="91"/>
+<wire x1="157.48" y1="50.8" x2="165.1" y2="50.8" width="0.1524" layer="91"/>
 <label x="160.02" y="50.8" size="1.778" layer="95"/>
 </segment>
@@
 <net name="LBO" class="0">
 <segment>
-<pinref part="U1" gate="G$1" pin="LBO"/>
-<wire x1="73.66" y1="50.8" x2="81.28" y2="50.8" width="0.1524" layer="91"/>
-<wire x1="81.28" y1="50.8" x2="81.28" y2="45.72" width="0.1524" layer="91"/>
 <wire x1="81.28" y1="45.72" x2="91.44" y2="45.72" width="0.1524" layer="91"/>
 <pinref part="T1" gate="G$1" pin="B"/>
@@
 <junction x="134.62" y="27.94"/>
 </segment>
-</net>
+<segment>
+<pinref part="U1" gate="G$1" pin="LBO"/>
+<wire x1="73.66" y1="50.8" x2="76.2" y2="50.8" width="0.1524" layer="91"/>
+<label x="73.66" y="50.8" size="1.778" layer="95"/>
+</segment>
+</net>

Commit message: Cleanup for BOM upload
Parts:
- renumbered LED1 to LOW, LED2 to PWR, U$11 to SW2
Changed lines of the file:
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@@
 <part name="FID2" library="microbuilder" deviceset="FIDUCIAL" device="&quot;&quot;"/>
 <part name="U$19" library="microbuilder" deviceset="VBAT" device=""/>
-<part name="LED1" library="microbuilder" deviceset="LED" device="0805_NOOUTLINE" value="RED"/>
+<part name="LOW" library="microbuilder" deviceset="LED" device="0805_NOOUTLINE" value="RED"/>
 <part name="R20" library="microbuilder" deviceset="RESISTOR" device="0805_NOOUTLINE" value="1K"/>
-<part name="LED2" library="microbuilder" deviceset="LED" device="0805_NOOUTLINE" value="BLUE"/>
+<part name="PWR" library="microbuilder" deviceset="LED" device="0805_NOOUTLINE" value="BLUE"/>
 <part name="R5" library="microbuilder" deviceset="RESISTOR" device="0805_NOOUTLINE" value="1K"/>
 <part name="R13" library="microbuilder" deviceset="RESISTOR" device="0805_NOOUTLINE" value="200K"/>
@@
 <part name="S4" library="SparkFun-Switches" library_urn="urn:adsk.eagle:library:535" deviceset="MOMENTARY-SWITCH-SPST" device="-PTH-6.0MM" package3d_urn="urn:adsk.eagle:package:40163/1"/>
 <part name="CN1" library="microusb-amphenol-10118194-0001LF" deviceset="USB" device="MICRO_20329" value="microUSB"/>
-<part name="U$11" library="rightangleslideswitchspdt" deviceset="OS102011MA1QN1" device=""/>
+<part name="SW2" library="rightangleslideswitchspdt" deviceset="OS102011MA1QN1" device=""/>
 <part name="JP1" library="microbuilder" deviceset="HEADER-1X2" device="ROUND" value="JP1"/>
 </parts>
@@
 <instance part="FID2" gate="G$1" x="236.22" y="22.86"/>
 <instance part="U$19" gate="G$1" x="15.24" y="73.66"/>
-<instance part="LED1" gate="G$1" x="101.6" y="25.4" rot="R270"/>
+<instance part="LOW" gate="G$1" x="101.6" y="25.4" rot="R270"/>
 <instance part="R20" gate="G$1" x="101.6" y="35.56" rot="R90"/>
-<instance part="LED2" gate="G$1" x="121.92" y="83.82"/>
+<instance part="PWR" gate="G$1" x="121.92" y="83.82"/>
 <instance part="R5" gate="G$1" x="109.22" y="83.82"/>
 <instance part="R13" gate="G$1" x="43.18" y="91.44" rot="R270"/>
@@
 <instance part="S4" gate="G$1" x="220.98" y="58.42"/>
 <instance part="CN1" gate="G$1" x="83.82" y="147.32"/>
-<instance part="U$11" gate="G$1" x="185.42" y="58.42"/>
+<instance part="SW2" gate="G$1" x="185.42" y="58.42"/>
 <instance part="JP1" gate="G$1" x="269.24" y="116.84"/>
 </instances>
@@
 <wire x1="127" y1="83.82" x2="127" y2="81.28" width="0.1524" layer="91"/>
 <pinref part="U$14" gate="G$1" pin="GND"/>
-<pinref part="LED2" gate="G$1" pin="C"/>
+<pinref part="PWR" gate="G$1" pin="C"/>
 <wire x1="124.46" y1="83.82" x2="127" y2="83.82" width="0.1524" layer="91"/>
 </segment>
@@
 </segment>
 <segment>
-<pinref part="LED1" gate="G$1" pin="C"/>
+<pinref part="LOW" gate="G$1" pin="C"/>
 <pinref part="U$20" gate="G$1" pin="GND"/>
 </segment>
@@
 </segment>
 <segment>
-<pinref part="U$11" gate="G$1" pin="P$1"/>
+<pinref part="SW2" gate="G$1" pin="P$1"/>
 <pinref part="U$16" gate="G$1" pin="GND"/>
 <wire x1="147.32" y1="58.42" x2="147.32" y2="60.96" width="0.1524" layer="91"/>
@@
 </segment>
 <segment>
-<pinref part="U$11" gate="G$1" pin="P$3"/>
+<pinref part="SW2" gate="G$1" pin="P$3"/>
 <wire x1="157.48" y1="60.96" x2="157.48" y2="50.8" width="0.1524" layer="91"/>
 <wire x1="157.48" y1="50.8" x2="165.1" y2="50.8" width="0.1524" layer="91"/>
@@
 <net name="N$2" class="0">
 <segment>
-<pinref part="LED1" gate="G$1" pin="A"/>
+<pinref part="LOW" gate="G$1" pin="A"/>
 <pinref part="R20" gate="G$1" pin="1"/>
 </segment>
@@
 <wire x1="152.4" y1="50.8" x2="139.7" y2="50.8" width="0.1524" layer="91"/>
 <label x="139.7" y="50.8" size="1.778" layer="95"/>
-<pinref part="U$11" gate="G$1" pin="P$2"/>
+<pinref part="SW2" gate="G$1" pin="P$2"/>
 <wire x1="152.4" y1="60.96" x2="152.4" y2="50.8" width="0.1524" layer="91"/>
 </segment>
@@
 <segment>
 <pinref part="R5" gate="G$1" pin="2"/>
-<pinref part="LED2" gate="G$1" pin="A"/>
+<pinref part="PWR" gate="G$1" pin="A"/>
 <wire x1="114.3" y1="83.82" x2="116.84" y2="83.82" width="0.1524" layer="91"/>
 </segment>
